Commit message: Keep gripper level and prevent search servo stalls

File: urdf/robot.urdf (robot description, URDF)
Before this commit: robot mypalletizer_260_pi_sim, 15 links, 14 joints
Links:
- added link wrist_level_link, mass 0.08
Joints:
- added joint wrist_level_joint: type revolute, parent link4, child wrist_level_link, origin xyz= 0.044 0 0 rpy=0 0 0, axis 0 0 1, limit lower=-3.14 upper=3.14 effort=12 velocity=1.5
- joint joint5_to_joint4: origin xyz= 0.044 0 0 rpy=  1.5707963 0 0  -> xyz=0 0 0 rpy=  1.5707963 0 0 ; parent link4 -> wrist_level_link
